File: test-project/kiwi-pwr-in.kicad_pcb (KiCad board)
At the start: 4 copper layers, 99.2 x 52 mm, 115 parts, among them IC1 TPS3808G50QDBVRQ1, J1 PS_ON_OFF, J2 INP_POWER, J3 Master_Reset, J4 OUTPUT, J5 BATT_PLUG, Q1 BUK7J2R4, Q2 BSS138, Q3 BSS138, Q4 BSS138, U1 TPSM265R1V5SILR, U2 74LVC2G17GW-Q100H, U3 LTC4376HDHD-TRPBF, U4 74LVC1G74DC-Q100H, U5 INA233AIDGSR, U6 INA233AIDGSR

Commit message: Test project
Parts:
- removed A1, A2, A5, A7: L / NC / R, Jumper:SolderJumper-3_P1.3mm_Open_RoundedPad1.0x1.5mm
- removed A3, A4, A6, A8: NC, Jumper:SolderJumper-3_P1.3mm_Open_RoundedPad1.0x1.5mm
- added D14: GREEN, LED_SMD:LED_0805_2012Metric, F.Cu at (121.1, 111.2)
- added D15: GREEN, LED_SMD:LED_0805_2012Metric, F.Cu at (126.1, 111.1)
- added J6: BATT In, Connector_PinHeader_2.54mm:PinHeader_2x02_P2.54mm_Vertical, F.Cu at (117.3, 89.5)
- added JP5: BATLED, Jumper:SolderJumper-2_P1.3mm_Open_RoundedPad1.0x1.5mm, F.Cu at (121.1, 114.7)
- added JP7: PSLED, Jumper:SolderJumper-2_P1.3mm_Open_RoundedPad1.0x1.5mm, F.Cu at (126.1, 114.6)
- added R45: 5.6k, Resistor_SMD:R_0805_2012Metric, F.Cu at (121.1, 107.6)
- added R46: 5.6k, Resistor_SMD:R_0805_2012Metric, F.Cu at (126.1, 107.6)
- D2: moved to F.Cu
- J2: value INP_POWER -> PS In; footprint Connector_PinHeader_2.54mm:PinHeader_2x04_P2.54mm_Vertical -> Connector_PinHeader_2.54mm:PinHeader_2x02_P2.54mm_Vertical
- moved Q3 59.0 mm to (151.1, 115.1), turned to 180 degrees
- moved R41 58.7 mm to (153.7, 115.1), turned to -90 degrees
- moved Q4 54.1 mm to (151.1, 109.5), turned to 180 degrees
- moved R43 53.8 mm to (153.7, 109.6), turned to -90 degrees
- moved R42 53.2 mm to (149.6, 113.5), turned to 90 degrees
- moved R44 49.9 mm to (149.6, 111.1), turned to -90 degrees
- moved D12 32.7 mm to (150.2, 89.2), turned to 180 degrees
- moved D13 32.1 mm to (150.2, 92.8), turned to 180 degrees
- moved R38 29.5 mm to (148.2, 114.0), turned to -90 degrees
- moved R39 26.3 mm to (148.2, 110.5), turned to 90 degrees
- moved JP1 24.6 mm to (124.8, 78.3), turned to 180 degrees
- moved U6 23.1 mm to (123.8, 102.4)
- moved R13 22.7 mm to (138.7, 96.4)
- moved J1 15.9 mm to (131.0, 77.1), turned to -90 degrees
- moved C24 15.3 mm to (128.2, 102.5), turned to 90 degrees
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Connections:
- net +DiodeOR_OUT renamed +PWR
- net Net-(D12-A) renamed +PBATT
- J2 pad 1: +BATT -> -BATT
- J2 pad 3: +BATT -> -BATT
- J4 pad 1: -BATT -> /SCL_3V3
- J4 pad 10: (no net) -> +28V
- J4 pad 11: (no net) -> +28V
- J4 pad 12: (no net) -> +28V
- J4 pad 2: -BATT -> +3V3_PI
- J4 pad 3: -BATT -> /SDA_3V3
- J4 pad 5: +28V -> -BATT
- J4 pad 6: +28V -> -BATT
- J4 pad 7: +28V -> -BATT
- J4 pad 8: +28V -> -BATT
- J4 pad 9: (no net) -> +28V
- J5 pad 1: +BATT_SEN -> +BATT
- J5 pad 3: +BATT_SEN -> +BATT
- R37 pad 1: +BATT -> +VBATT
- R37 pad 2: +BATT_SEN -> +BATT
- U5 pad 1: /A1_BATT -> -BATT
- U5 pad 10: +BATT -> +VBATT
- U5 pad 2: /A0_BATT -> -BATT
- U5 pad 8: +BATT_SEN -> +BATT
- U5 pad 9: +BATT_SEN -> +BATT
- U6 pad 1: /A1_PS -> -BATT
- U6 pad 2: /A0_PS -> +5V
Routing:
- net /SCL_5V: track 0.00 -> 88.3 mm, vias 0 -> 2
- net /SDA_5V: track 0.00 -> 77.3 mm
- net +PBATT: track 0.00 -> 49.9 mm
- net +PWR: track 18.9 -> 48.1 mm, vias 2 -> 4
- net +5V: track 66.8 -> 43.6 mm, vias 9 -> 16
- net +PS_SEN: track 0.00 -> 16.3 mm, vias 0 -> 2
- net +3V3_PI: track 0.00 -> 14.8 mm
- net /SDA_3V3: track 0.00 -> 14.0 mm
- net /VSS: track 25.6 -> 37.9 mm, vias 1 -> 0
- net /~{DOR_ON}: track 10.9 -> 22.1 mm
- net /~{DOR_OFF}: track 21.5 -> 32.0 mm
- net -BATT: track 0.00 -> 8.64 mm, vias 201 -> 337
- net +BATT: track 0.00 -> 7.27 mm
- net /SCL_3V3: track 0.00 -> 7.09 mm
- net +PS: track 0.00 -> 6.67 mm
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- added copper zone on In2.Cu, net +5V
- added copper zone on F.Cu, net +BATT
- added copper zone on F.Cu, net +PBATT
- added copper zone on F.Cu, net +PS
- added copper zone on F.Cu, net +PS_SEN
- added copper zone on F.Cu, net +VBATT
Other:
- board text added: "BAT IN"
- board text added: "BATT EN"
- board text added: "BATT PWR IN"
- board text added: "PS IN"
- board text added: "PS PWR IN"
- board text removed: "+28V"
