File: test-project/kiwi-pwr-in.kicad_sch (KiCad schematic)
At the start: 115 parts, among them IC1 TPS3808G50QDBVRQ1, J1 PS_ON_OFF, J2 INP_POWER, J3 Master_Reset, J4 OUTPUT, J5 BATT_PLUG, Q1 BUK7J2R4, Q2 BSS138, Q3 BSS138, Q4 BSS138, U1 TPSM265R1V5SILR, U2 74LVC2G17GW-Q100H, U3 LTC4376HDHD-TRPBF, U4 74LVC1G74DC-Q100H, U5 INA233AIDGSR, U6 INA233AIDGSR

Commit message: Test project
Parts:
- removed A1, A2, A5, A7: L / NC / R, Jumper:SolderJumper-3_P1.3mm_Open_RoundedPad1.0x1.5mm, symbol Jumper:SolderJumper_3_Open
- removed A3, A4, A6, A8: NC, Jumper:SolderJumper-3_P1.3mm_Open_RoundedPad1.0x1.5mm, symbol Jumper:SolderJumper_3_Open
- removed J2: INP_POWER, Connector_PinHeader_2.54mm:PinHeader_2x04_P2.54mm_Vertical, symbol Connector_Generic:Conn_02x04_Odd_Even
- added D14, D15: GREEN, LED_SMD:LED_0805_2012Metric, symbol Device:LED
- added J2: PS In, Connector_PinHeader_2.54mm:PinHeader_2x02_P2.54mm_Vertical, symbol Connector_Generic:Conn_02x02_Odd_Even
- added J6: BATT In, Connector_PinHeader_2.54mm:PinHeader_2x02_P2.54mm_Vertical, symbol Connector_Generic:Conn_02x02_Odd_Even
- added JP5: BATLED, Jumper:SolderJumper-2_P1.3mm_Open_RoundedPad1.0x1.5mm, symbol Jumper:SolderJumper_2_Open
- added JP7: PSLED, Jumper:SolderJumper-2_P1.3mm_Open_RoundedPad1.0x1.5mm, symbol Jumper:SolderJumper_2_Open
- added R45, R46: 5.6k, Resistor_SMD:R_0805_2012Metric, symbol Device:R_Small_US
- J4: symbol Connector_Generic:Conn_02x04_Odd_Even -> Connector_Generic:Conn_02x06_Odd_Even
- J5: now not fitted; now left out of the parts list
Connections:
- net +BATT_SEN is gone; now on net +BATT: J5.1 (Pin_1), J5.3 (Pin_3), R37.2, U5.8 (Vbus), U5.9 (Vin-)
- net A0_BATT is gone; now on net -BATT: U5.2 (A0)
- net A0_PS is gone; now on net +5V: U6.2 (A0)
- net A1_BATT is gone; now on net -BATT: U5.1 (A1)
- net A1_PS is gone; now on net -BATT: U6.1 (A1)
- net +28V: now also J4.10 (Pin_10), J4.11 (Pin_11), J4.12 (Pin_12), J4.9 (Pin_9); no longer J4.5 (Pin_5), J4.6 (Pin_6), J4.7 (Pin_7), J4.8 (Pin_8)
- net +3V3_PI: now also J4.2 (Pin_2)
- net +BATT: no longer R37.1, U5.10 (Vin+)
- net +PS: now also J2.2 (Pin_2), J2.4 (Pin_4)
- net +PS_SEN: now also R46.1
- net -BATT: now also J4.5 (Pin_5), J4.6 (Pin_6), J4.7 (Pin_7), J4.8 (Pin_8), J2.1 (Pin_1), J2.3 (Pin_3), J6.1 (Pin_1), J6.3 (Pin_3), JP5.1 (A), JP7.1 (A); no longer J4.1 (Pin_1), J4.2 (Pin_2), J4.3 (Pin_3)
- net SCL_3V3: now also J4.1 (Pin_1)
- net SDA_3V3: now also J4.3 (Pin_3)
- net +PBATT: now reaches D12.2 (A), J5.2 (Pin_2), J5.4 (Pin_4)
- net +PBATT: now also R45.1
- net +DiodeOR_OUT renamed +PWR
- new net: D14.2 (A), R45.2
- new net: D15.2 (A), R46.2
- new net: D15.1 (K), JP7.2 (B)
- new net: D14.1 (K), JP5.2 (B)
- new net +VBATT: J6.2 (Pin_2), J6.4 (Pin_4), R37.1, U5.10 (Vin+)
Other:
- note added: "(RTM) R11 & C7 are for in-rush control Leave unpopulated if not required R35 and R36 are experiments to eliminate brief moment on when the batt/ps is enabled R12 & R36 needs to be very close to Q1 gate"
- note added: "Addressing: Base: 0b0100_[A1][A0] A -> GND: 0b00 A -> VCC: 0b01 A -> SDA: 0b10 A -> SCL: 0b11 Selected: 0b0100_0000"
- note added: "Addressing: Base: 0b0100_[A1][A0] A -> GND: 0b00 A -> VCC: 0b01 A -> SDA: 0b10 A -> SCL: 0b11 Selected: 0b0100_0001"
- note added: "C20 DNP Unless +VBATT Noisy"
- note removed: "(RTM) R11 & C7 are for in-rush control Leave unpopulated if not required R35 and R36 are experimnets to eliminate brief moment on when the batt/ps is enabled R12 & R36 needs to be very close to Q1 gate"
- note removed: "Addressing: Base: 0b0100_[A1][A0] A -> GND: 0b00 A -> VCC: 0b01 A -> SDA: 0b10 A -> SCL: 0b11"
- note removed: "C20 DNP Unless +BATT Noisy"
- note removed: "Use A1 ONLY IF not present at input"
- moved on the sheet: D12, D13

Commit message: BOM
Parts:
- C10, C24: Last Checked (none) -> 2026-08-09T03:01:00.990148+00:00; Mfr (none) -> KYOCERA AVX; Mfr # (none) -> 08055C104J4T4A; Mouser (none) -> https://www.mouser.com/en/ProductDetail/KYOCERA-AVX/08055C1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; Mouser # (none) -> 581-08055C104J4T4A; Mouser Lifecycle (none) -> Unknown; Mouser Price Breaks (Raw) (none) -> 1:0.18|10:0.074|100:0.065|500:0.049|1000:0.044|2500:0.039|5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; Mouser Qty/Price (none) -> 1:$0.18 | 10:$0.07 | 100:$0.07 | 500:$0.05; Mouser Stock (none) -> 11201 In Stock; Mouser Stock Qty (none) -> 11201; Vendor Description (none) -> Multilayer Ceramic Capacitors MLCC - SMD/SMT KAM21BR71H104J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
- C11, C12, C13, C14, C15, C16, C17, C18: Last Checked (none) -> 2026-08-09T03:01:00.990148+00:00; Mfr (none) -> TDK; Mfr # (none) -> CGA9P3X7S2A156M250KB; Mouser (none) -> https://www.mouser.com/en/ProductDetail/TDK/CGA9P3X7S2A156M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; Mouser # (none) -> 810-CGA9P3X7S2A156M; Mouser Lifecycle (none) -> Unknown; Mouser Price Breaks (Raw) (none) -> 1:3.14|10:2.18|50:1.8|100:1.69|500:1.4|1000:1.32; Mouser Qty/Price (none) -> 1:$3.14 | 10:$2.18 | 50:$1.80 | 100:$1.69; Mouser Stock (none) -> 25873 In Stock; Mouser Stock Qty (none) -> 25873; Vendor Description (none) -> Multilayer Ceramic Capacitors MLCC - SMD/SMT CGA 2220 100V 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
- C19: DigiKey (none) -> https://www.digikey.com/en/products/detail/kyocera-avx/KAM0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; DigiKey # (none) -> 478-KAM05CR71A105KHCT-ND; DigiKey Lifecycle (none) -> Active; DigiKey Price Breaks (Raw) (none) -> 1:0.17|10:0.099|50:0.0702|100:0.0613|500:0.04634; DigiKey Qty/Price (none) -> 1:$0.17 | 10:$0.10 | 50:$0.07 | 100:$0.06; DigiKey Stock (none) -> 6 in stock; DigiKey Stock Qty (none) -> 6; Last Checked (none) -> 2026-08-09T03:01:00.990148+00:00; Mfr (none) -> KYOCERA AVX; Mfr # (none) -> KAM05CR71A105KH; Mouser (none) -> https://www.mouser.com/en/ProductDetail/KYOCERA-AVX/KAM05CR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; Mouser # (none) -> 581-KAM05CR71A105KH; Mouser Lifecycle (none) -> Unknown; Mouser Price Breaks (Raw) (none) -> 1:0.19|10:0.118|100:0.071|500:0.056|1000:0.051|2500:0.045|5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; Mouser Qty/Price (none) -> 1:$0.19 | 10:$0.12 | 100:$0.07 | 500:$0.06; Mouser Stock (none) -> Availability unknown; Mouser Stock Qty (none) -> 0; Vendor Description (none) -> 1 µF ±10% 10V Ceramic Capacitor X7R 0402 (1005 Metric)
- C2: Last Checked (none) -> 2026-08-09T03:01:00.990148+00:00; Mfr (none) -> Murata Electronics; Mfr # (none) -> GCM31CC72A225KE02L; Mouser (none) -> https://www.mouser.com/en/ProductDetail/Murata-Electronics/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; Mouser # (none) -> 81-GCM31CC72A225KE2L; Mouser Lifecycle (none) -> Unknown; Mouser Price Breaks (Raw) (none) -> 1:0.63|10:0.31|100:0.272|500:0.233|1000:0.218|2000:0.192|40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; Mouser Qty/Price (none) -> 1:$0.63 | 10:$0.31 | 100:$0.27 | 500:$0.23; Mouser Stock (none) -> 26577 In Stock; Mouser Stock Qty (none) -> 26577; Vendor Description (none) -> Multilayer Ceramic Capacitors MLCC - SMD/SMT 2.2 uF 100 VDC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
- C20, C22, C3, C4, C5, C8: Last Checked (none) -> 2026-08-09T03:01:00.990148+00:00; Mfr (none) -> KEMET; Mfr # (none) -> C0402C104K4RACAUTO7411; Mouser (none) -> https://www.mouser.com/en/ProductDetail/KEMET/C0402C104K4RA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; Mouser # (none) -> 80-C0402C104K4RAUTLR; Mouser Lifecycle (none) -> Unknown; Mouser Price Breaks (Raw) (none) -> 1:0.13|10:0.054|100:0.032|500:0.025|1000:0.024|50000:0.024; Mouser Qty/Price (none) -> 1:$0.13 | 10:$0.05 | 100:$0.03 | 500:$0.03; Mouser Stock (none) -> 80862 In Stock; Mouser Stock Qty (none) -> 80862; Vendor Description (none) -> Multilayer Ceramic Capacitors MLCC - SMD/SMT 16V 0.1uF X7R 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
- C21: Last Checked (none) -> 2026-08-09T03:01:00.990148+00:00; Mfr (none) -> YAGEO; Mfr # (none) -> AC0805KFX7R8BB474; Mouser (none) -> https://www.mouser.com/en/ProductDetail/YAGEO/AC0805KFX7R8B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; Mouser # (none) -> 603-AC805KFX7R8BB474; Mouser Lifecycle (none) -> Unknown; Mouser Price Breaks (Raw) (none) -> 1:0.25|10:0.106|100:0.093|500:0.072|1000:0.066|2500:0.059|5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; Mouser Qty/Price (none) -> 1:$0.25 | 10:$0.11 | 100:$0.09 | 500:$0.07; Mouser Stock (none) -> 9946 In Stock; Mouser Stock Qty (none) -> 9946; Vendor Description (none) -> Multilayer Ceramic Capacitors MLCC - SMD/SMT 25V 0.47uF X7R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
- C23: Last Checked (none) -> 2026-08-09T03:01:00.990148+00:00; Mfr (none) -> KYOCERA AVX; Mfr # (none) -> 08051C474K4T2A; Mouser (none) -> https://www.mouser.com/en/ProductDetail/KYOCERA-AVX/08051C4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; Mouser # (none) -> 581-08051C474K4T2A; Mouser Lifecycle (none) -> Unknown; Mouser Price Breaks (Raw) (none) -> 1:0.31|10:0.299|2000:0.299|4000:0.207; Mouser Qty/Price (none) -> 1:$0.31 | 10:$0.30 | 2000:$0.30 | 4000:$0.21; Mouser Stock (none) -> 20923 In Stock; Mouser Stock Qty (none) -> 20923; Vendor Description (none) -> Multilayer Ceramic Capacitors MLCC - SMD/SMT KAM21KR72A474K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
- C6: Last Checked (none) -> 2026-08-09T03:01:00.990148+00:00; Mfr (none) -> Murata Electronics; Mfr # (none) -> GRM32ER71E226ME15L; Mouser (none) -> https://www.mouser.com/en/ProductDetail/Murata-Electronics/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; Mouser # (none) -> 81-GRM32ER71E226ME5L; Mouser Lifecycle (none) -> End of Life; Mouser Price Breaks (Raw) (none) -> 1:0.78|10:0.376|100:0.34|500:0.28|1000:0.247|2000:0.226; Mouser Qty/Price (none) -> 1:$0.78 | 10:$0.38 | 100:$0.34 | 500:$0.28; Mouser Stock (none) -> 1646 In Stock; Mouser Stock Qty (none) -> 1646; Vendor Description (none) -> Multilayer Ceramic Capacitors MLCC - SMD/SMT 22 uF 25 VDC 2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
- C9: Last Checked (none) -> 2026-08-09T03:01:00.990148+00:00; Mfr (none) -> TDK; Mfr # (none) -> CGA4J3X7R1H155K125AB; Mouser (none) -> https://www.mouser.com/en/ProductDetail/TDK/CGA4J3X7R1H155K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; Mouser # (none) -> 810-CGA4J3X7R1H155KB; Mouser Lifecycle (none) -> Unknown; Mouser Price Breaks (Raw) (none) -> 1:0.37|10:0.165|100:0.147|500:0.116|1000:0.107|2000:0.095|4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; Mouser Qty/Price (none) -> 1:$0.37 | 10:$0.17 | 100:$0.15 | 500:$0.12; Mouser Stock (none) -> 7563 In Stock; Mouser Stock Qty (none) -> 7563; Vendor Description (none) -> Multilayer Ceramic Capacitors MLCC - SMD/SMT CGA 0805 50V 1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
- D1: Last Checked (none) -> 2026-08-09T03:01:00.990148+00:00; Mfr (none) -> Littelfuse; Mfr # (none) -> SMAJ40A; Mouser (none) -> https://www.mouser.com/en/ProductDetail/Littelfuse/SMAJ40A?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; Mouser # (none) -> 576-SMAJ40A; Mouser Lifecycle (none) -> Unknown; Mouser Price Breaks (Raw) (none) -> 1:0.38|10:0.208|100:0.175|500:0.135|1000:0.117|2500:0.098|5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; Mouser Qty/Price (none) -> 1:$0.38 | 10:$0.21 | 100:$0.17 | 500:$0.14; Mouser Stock (none) -> 42488 In Stock; Mouser Stock Qty (none) -> 42488; Vendor Description (none) -> ESD Protection Diodes / TVS Diodes 400W 40V 5% Uni-Directio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
- D10: DigiKey (none) -> https://www.digikey.com/en/products/detail/yageo/ES1B/20415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; DigiKey # (none) -> 13-ES1BCT-ND; DigiKey Lifecycle (none) -> Active; DigiKey Price Breaks (Raw) (none) -> 1:0.34|10:0.208|50:0.149|100:0.1298|500:0.09588; DigiKey Qty/Price (none) -> 1:$0.34 | 10:$0.21 | 50:$0.15 | 100:$0.13; DigiKey Stock (none) -> 1305 in stock; DigiKey Stock Qty (none) -> 1305; Last Checked (none) -> 2026-08-09T03:01:00.990148+00:00; Mfr (none) -> YAGEO; Mfr # (none) -> ES1B; Vendor Description (none) -> Diode 100 V 1A Surface Mount DO-214AC (SMA)
- D11, D9: DigiKey (none) -> https://www.digikey.com/en/products/detail/diotec-semicondu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; DigiKey # (none) -> 4878-1N4148WGWCT-ND; DigiKey Lifecycle (none) -> Active; DigiKey Price Breaks (Raw) (none) -> 1:0.1|10:0.057|50:0.04|100:0.0346|500:0.02478; DigiKey Qty/Price (none) -> 1:$0.10 | 10:$0.06 | 50:$0.04 | 100:$0.03; DigiKey Stock (none) -> 24163 in stock; DigiKey Stock Qty (none) -> 24163; Last Checked (none) -> 2026-08-09T03:01:00.990148+00:00; Mfr (none) -> Diotec Semiconductor; Mfr # (none) -> 1N4148WGW; Vendor Description (none) -> Diode 75 V 150mA Surface Mount SOD-123
- D12, D13: DigiKey (none) -> https://www.digikey.com/en/products/detail/taiwan-semicondu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; DigiKey # (none) -> 1801-TSSA5U60HCT-ND; DigiKey Lifecycle (none) -> Active; DigiKey Price Breaks (Raw) (none) -> 1:0.7|10:0.432|50:0.3144|100:0.2762|500:0.20876; DigiKey Qty/Price (none) -> 1:$0.70 | 10:$0.43 | 50:$0.31 | 100:$0.28; DigiKey Stock (none) -> 13127 in stock; DigiKey Stock Qty (none) -> 13127; Last Checked (none) -> 2026-08-09T03:01:00.990148+00:00; Mfr (none) -> Taiwan Semiconductor Corporation; Mfr # (none) -> TSSA5U60H; Vendor Description (none) -> Diode 60 V 5A Surface Mount DO-214AC (SMA)
- D14, D15: DigiKey (none) -> https://www.digikey.com/en/products/detail/rohm-semiconduct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; DigiKey # (none) -> 846-SMLMN2ECTT86CCT-ND; DigiKey Lifecycle (none) -> Active; DigiKey Price Breaks (Raw) (none) -> 1:0.75|10:0.521|100:0.3792|500:0.31586|1000:0.29509; DigiKey Qty/Price (none) -> 1:$0.75 | 10:$0.52 | 100:$0.38 | 500:$0.32; DigiKey Stock (none) -> 804 in stock; DigiKey Stock Qty (none) -> 804; Last Checked (none) -> 2026-08-09T03:01:00.990148+00:00; Mfr (none) -> Rohm Semiconductor; Mfr # (none) -> SMLMN2ECTT86C; Vendor Description (none) -> Green 527nm LED Indication - Discrete 3V 0805 (2012 Metric)
- D2: DigiKey (none) -> https://www.digikey.com/en/products/detail/würth-elektronik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; DigiKey # (none) -> 732-SMAJ24ACT-ND; DigiKey Lifecycle (none) -> Active; DigiKey Price Breaks (Raw) (none) -> 1:0.29|10:0.269|100:0.241|500:0.21; DigiKey Qty/Price (none) -> 1:$0.29 | 10:$0.27 | 100:$0.24 | 500:$0.21; DigiKey Stock (none) -> 10565 in stock; DigiKey Stock Qty (none) -> 10565; Last Checked (none) -> 2026-08-09T03:01:00.990148+00:00; Mfr (none) -> Würth Elektronik; Mfr # (none) -> SMAJ24A; Mouser (none) -> https://www.mouser.com/en/ProductDetail/YAGEO/SMAJ24A-TR7?q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; Mouser # (none) -> 603-SMAJ24A/TR7; Mouser Lifecycle (none) -> Unknown; Mouser Price Breaks (Raw) (none) -> 1:0.37|10:0.161|100:0.141|500:0.104|1000:0.092|2000:0.068|5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; Mouser Qty/Price (none) -> 1:$0.37 | 10:$0.16 | 100:$0.14 | 500:$0.10; Mouser Stock (none) -> 1540 In Stock; Mouser Stock Qty (none) -> 1540; Vendor Description (none) -> 38.9V Clamp 10.3A Ipp Tvs Diode Surface Mount DO-214AC
- D3, D8: DigiKey (none) -> https://www.digikey.com/en/products/detail/rohm-semiconduct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; DigiKey # (none) -> 846-SMLMN2ECTT86CTR-ND; DigiKey Lifecycle (none) -> Active; DigiKey Price Breaks (Raw) (none) -> 3000:0.26838|6000:0.25478|9000:0.24781|15000:0.23994|21000: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; DigiKey Qty/Price (none) -> 3000:$0.27 | 6000:$0.25 | 9000:$0.25 | 15000:$0.24; DigiKey Stock (none) -> 804 in stock; DigiKey Stock Qty (none) -> 804; Last Checked (none) -> 2026-08-09T03:01:00.990148+00:00; Mfr (none) -> ROHM Semiconductor; Mfr # (none) -> SMLMN2ECTT86C; Mouser (none) -> https://www.mouser.com/en/ProductDetail/ROHM-Semiconductor/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; Mouser # (none) -> 755-SMLMN2ECTT86C; Mouser Lifecycle (none) -> Unknown; Mouser Price Breaks (Raw) (none) -> 1:0.73|10:0.506|100:0.369|500:0.308|1000:0.288|3000:0.264|6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; Mouser Qty/Price (none) -> 1:$0.73 | 10:$0.51 | 100:$0.37 | 500:$0.31; Mouser Stock (none) -> 724 In Stock; Mouser Stock Qty (none) -> 724; Vendor Description (none) -> Single Color LEDs Add PTC 5-0617-50 AECQ-102
- D4: Last Checked (none) -> 2026-08-09T03:01:00.990148+00:00; Mfr (none) -> Diodes Incorporated; Mfr # (none) -> DDZ9699T-7; Mouser (none) -> https://www.mouser.com/en/ProductDetail/Diodes-Incorporated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; Mouser # (none) -> 621-DDZ9699T-7; Mouser Lifecycle (none) -> Unknown; Mouser Price Breaks (Raw) (none) -> 1:0.51|10:0.235|100:0.193|500:0.174|1000:0.158|3000:0.158; Mouser Qty/Price (none) -> 1:$0.51 | 10:$0.23 | 100:$0.19 | 500:$0.17; Mouser Stock (none) -> 7675 In Stock; Mouser Stock Qty (none) -> 7675; Vendor Description (none) -> Zener Diodes 150MW 12V
- D5: Last Checked (none) -> 2026-08-09T03:01:00.990148+00:00; Mfr (none) -> ROHM Semiconductor; Mfr # (none) -> SML-H12U8TT86C; Mouser (none) -> https://www.mouser.com/en/ProductDetail/ROHM-Semiconductor/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; Mouser # (none) -> 755-SML-H12U8TT86C; Mouser Lifecycle (none) -> Unknown; Mouser Price Breaks (Raw) (none) -> 1:0.31|10:0.213|100:0.15|500:0.122|1000:0.11|3000:0.099|600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; Mouser Qty/Price (none) -> 1:$0.31 | 10:$0.21 | 100:$0.15 | 500:$0.12; Mouser Stock (none) -> 12678 In Stock; Mouser Stock Qty (none) -> 12678; Vendor Description (none) -> Single Color LEDs The factory is currently not accepting or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
- D6, D7: Last Checked (none) -> 2026-08-09T03:01:00.990148+00:00; Mfr (none) -> Panjit; Mfr # (none) -> BAT54C-AU_R1_000A1; Mouser (none) -> https://www.mouser.com/en/ProductDetail/Panjit/BAT54C-AU_R1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; Mouser # (none) -> 241-BAT54C-AUR1000A1; Mouser Lifecycle (none) -> Unknown; Mouser Price Breaks (Raw) (none) -> 1:0.19|10:0.118|100:0.074|500:0.06|1000:0.052|3000:0.045|60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; Mouser Qty/Price (none) -> 1:$0.19 | 10:$0.12 | 100:$0.07 | 500:$0.06; Mouser Stock (none) -> 3073 In Stock; Mouser Stock Qty (none) -> 3073; Vendor Description (none) -> Schottky Diodes & Rectifiers 30V,Schottky,SOT-23,0.2A
- IC1: DigiKey (none) -> https://www.digikey.com/en/products/detail/texas-instrument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; DigiKey # (none) -> 296-23126-1-ND; DigiKey Lifecycle (none) -> Active; DigiKey Price Breaks (Raw) (none) -> 1:2.33|10:1.727|25:1.5756|100:1.4094|250:1.33024|500:1.29132; DigiKey Qty/Price (none) -> 1:$2.33 | 10:$1.73 | 25:$1.58 | 100:$1.41; DigiKey Stock (none) -> 0 in stock; DigiKey Stock Qty (none) -> 0; Last Checked (none) -> 2026-08-09T03:01:00.990148+00:00; Mfr (none) -> Texas Instruments; Mfr # (none) -> TPS3808G50QDBVRQ1; Vendor Description (none) -> Supervisor Open Drain or Open Collector 1 Channel SOT-23-6
- J1, J3, JP1: Last Checked (none) -> 2026-08-09T03:15:47.868936+00:00
- J4: DigiKey (none) -> https://www.digikey.com/en/products/detail/amphenol-cs-fci/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; DigiKey Lifecycle (none) -> Active; DigiKey Price Breaks (Raw) (none) -> 1:2.67|10:2.271|100:1.9297; DigiKey Qty/Price (none) -> 1:$2.67 | 10:$2.27 | 100:$1.93; DigiKey Stock (none) -> 8712 in stock; DigiKey Stock Qty (none) -> 8712; Last Checked (none) -> 2026-08-09T03:01:00.990148+00:00; Mfr Amphenol ICC -> Amphenol ICC (FCI); Vendor Description (none) -> 20 Position Receptacle Connector 0.050" (1.27mm) Surface Mo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
- L1: DigiKey (none) -> https://www.digikey.com/en/products/detail/bourns-inc/SRR12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; DigiKey # (none) -> SRR1260A-2R2YCT-ND; DigiKey Lifecycle (none) -> Active; DigiKey Price Breaks (Raw) (none) -> 1:1.3|10:1.066|25:0.986|50:0.9294|100:0.8763|250:0.81072; DigiKey Qty/Price (none) -> 1:$1.30 | 10:$1.07 | 25:$0.99 | 50:$0.93; DigiKey Stock (none) -> 262 in stock; DigiKey Stock Qty (none) -> 262; Last Checked (none) -> 2026-08-09T03:01:00.990148+00:00; Mfr (none) -> Bourns Inc.; Mfr # (none) -> SRR1260A-2R2Y; Vendor Description (none) -> 2.2 µH Shielded Drum Core, Wirewound Inductor 8.2 A 10.5mOh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
- Q1: DigiKey (none) -> https://www.digikey.com/en/products/detail/nexperia-usa-inc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; DigiKey # (none) -> 1727-BUK7J2R4-80MXCT-ND; DigiKey Lifecycle (none) -> Active; DigiKey Price Breaks (Raw) (none) -> 1:3.61|10:2.356|50:1.8138|100:1.6392|500:1.3331; DigiKey Qty/Price (none) -> 1:$3.61 | 10:$2.36 | 50:$1.81 | 100:$1.64; DigiKey Stock (none) -> 1407 in stock; DigiKey Stock Qty (none) -> 1407; Last Checked (none) -> 2026-08-09T03:01:00.990148+00:00; Mfr (none) -> Nexperia USA Inc.; Mfr # (none) -> BUK7J2R4-80MX; Vendor Description (none) -> N-Channel 80 V 231A (Ta) 294W (Ta) Surface Mount LFPAK56, P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
- Q2, Q3, Q4: DigiKey (none) -> https://www.digikey.com/en/products/detail/nexperia-usa-inc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; DigiKey # (none) -> 1727-1142-1-ND; DigiKey Lifecycle (none) -> Active; DigiKey Price Breaks (Raw) (none) -> 1:0.19|10:0.119|50:0.0848|100:0.0735|500:0.05348; DigiKey Qty/Price (none) -> 1:$0.19 | 10:$0.12 | 50:$0.08 | 100:$0.07; DigiKey Stock (none) -> 74456 in stock; DigiKey Stock Qty (none) -> 74456; Last Checked (none) -> 2026-08-09T03:01:00.990148+00:00; Mfr (none) -> Nexperia USA Inc.; Mfr # (none) -> BSS138P,215; Vendor Description (none) -> N-Channel 60 V 360mA (Ta) 350mW (Ta), 1.14W (Tc) Surface Mo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
- R1, R16, R2, R30: DigiKey (none) -> https://www.digikey.com/en/products/detail/vishay-dale/CRCW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; DigiKey # (none) -> 541-100KLCT-ND; DigiKey Lifecycle (none) -> Active; DigiKey Price Breaks (Raw) (none) -> 1:0.1|10:0.032|25:0.0236|50:0.0192|100:0.0157|250:0.01228|5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; DigiKey Qty/Price (none) -> 1:$0.10 | 10:$0.03 | 25:$0.02 | 50:$0.02; DigiKey Stock (none) -> 4115632 in stock; DigiKey Stock Qty (none) -> 4115632; Last Checked (none) -> 2026-08-09T03:01:00.990148+00:00; Mfr (none) -> Vishay Dale; Mfr # (none) -> CRCW0402100KFKED; Mouser (none) -> https://www.mouser.com/en/ProductDetail/Vishay/CRCW0402100K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; Mouser # (none) -> 71-CRCW0402-100K-E3; Mouser Lifecycle (none) -> Unknown; Mouser Price Breaks (Raw) (none) -> 1:0.1|10:0.02|100:0.016|250:0.013|500:0.011|1000:0.009|5000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; Mouser Qty/Price (none) -> 1:$0.10 | 10:$0.02 | 100:$0.02 | 250:$0.01; Mouser Replacement (none) -> 71-CRCW0402-100K; Mouser Stock (none) -> 2923962 In Stock; Mouser Stock Qty (none) -> 2923962; Vendor Description (none) -> 100 kOhms ±1% 0.063W, 1/16W Chip Resistor 0402 (1005 Metric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
- R10, R13, R34: DigiKey (none) -> https://www.digikey.com/en/products/detail/vishay-dale/CRCW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; DigiKey # (none) -> 541-1.00KCCT-ND; DigiKey Lifecycle (none) -> Active; DigiKey Price Breaks (Raw) (none) -> 1:0.1|10:0.044|25:0.0332|50:0.0272|100:0.0225|250:0.01796|5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; DigiKey Qty/Price (none) -> 1:$0.10 | 10:$0.04 | 25:$0.03 | 50:$0.03; DigiKey Stock (none) -> 1347365 in stock; DigiKey Stock Qty (none) -> 1347365; Last Checked (none) -> 2026-08-09T03:01:00.990148+00:00; Mfr (none) -> Vishay Dale; Mfr # (none) -> CRCW08051K00FKEA; Mouser (none) -> https://www.mouser.com/en/ProductDetail/Vishay/CRCW08051K00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; Mouser # (none) -> 71-CRCW0805-1.0K-E3; Mouser Lifecycle (none) -> Unknown; Mouser Price Breaks (Raw) (none) -> 1:0.1|10:0.028|100:0.023|250:0.018|500:0.016|1000:0.014|500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; Mouser Qty/Price (none) -> 1:$0.10 | 10:$0.03 | 100:$0.02 | 250:$0.02; Mouser Replacement (none) -> 71-CRCW0805-1.0K; Mouser Stock (none) -> 468345 In Stock; Mouser Stock Qty (none) -> 468345; Vendor Description (none) -> 1 kOhms ±1% 0.125W, 1/8W Chip Resistor 0805 (2012 Metric) A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
Commit message: Preference
Parts:
- C10, C24: Last Checked 2026-08-09T03:01:00.990148+00:00 -> (none); Mfr KYOCERA AVX -> (none); Mfr # 08055C104J4T4A -> (none); Mouser https://www.mouser.com/en/ProductDetail/KYOCERA-AVX/08055C1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 -> (none); Mouser # 581-08055C104J4T4A -> (none); Mouser Lifecycle Unknown -> (none); Mouser Price Breaks (Raw) 1:0.18|10:0.074|100:0.065|500:0.049|1000:0.044|2500:0.039|5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 -> (none); Mouser Qty/Price 1:$0.18 | 10:$0.07 | 100:$0.07 | 500:$0.05 -> (none); Mouser Stock 11201 In Stock -> (none); Mouser Stock Qty 11201 -> (none); Vendor Description Multilayer Ceramic Capacitors MLCC - SMD/SMT KAM21BR71H104J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 -> (none)
- C11, C12, C13, C14, C15, C16, C17, C18: Last Checked 2026-08-09T03:01:00.990148+00:00 -> (none); Mfr TDK -> (none); Mfr # CGA9P3X7S2A156M250KB -> (none); Mouser https://www.mouser.com/en/ProductDetail/TDK/CGA9P3X7S2A156M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 -> (none); Mouser # 810-CGA9P3X7S2A156M -> (none); Mouser Lifecycle Unknown -> (none); Mouser Price Breaks (Raw) 1:3.14|10:2.18|50:1.8|100:1.69|500:1.4|1000:1.32 -> (none); Mouser Qty/Price 1:$3.14 | 10:$2.18 | 50:$1.80 | 100:$1.69 -> (none); Mouser Stock 25873 In Stock -> (none); Mouser Stock Qty 25873 -> (none); Vendor Description Multilayer Ceramic Capacitors MLCC - SMD/SMT CGA 2220 100V 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 -> (none)
- C19: DigiKey https://www.digikey.com/en/products/detail/kyocera-avx/KAM0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 -> (none); DigiKey # 478-KAM05CR71A105KHCT-ND -> (none); DigiKey Lifecycle Active -> (none); DigiKey Price Breaks (Raw) 1:0.17|10:0.099|50:0.0702|100:0.0613|500:0.04634 -> (none); DigiKey Qty/Price 1:$0.17 | 10:$0.10 | 50:$0.07 | 100:$0.06 -> (none); DigiKey Stock 6 in stock -> (none); DigiKey Stock Qty 6 -> (none); Last Checked 2026-08-09T03:01:00.990148+00:00 -> (none); Mfr KYOCERA AVX -> (none); Mfr # KAM05CR71A105KH -> (none); Mouser https://www.mouser.com/en/ProductDetail/KYOCERA-AVX/KAM05CR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 -> (none); Mouser # 581-KAM05CR71A105KH -> (none); Mouser Lifecycle Unknown -> (none); Mouser Price Breaks (Raw) 1:0.19|10:0.118|100:0.071|500:0.056|1000:0.051|2500:0.045|5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 -> (none); Mouser Qty/Price 1:$0.19 | 10:$0.12 | 100:$0.07 | 500:$0.06 -> (none); Mouser Stock Availability unknown -> (none); Mouser Stock Qty 0 -> (none); Vendor Description 1 µF ±10% 10V Ceramic Capacitor X7R 0402 (1005 Metric) -> (none)
- C2: Last Checked 2026-08-09T03:01:00.990148+00:00 -> (none); Mfr Murata Electronics -> (none); Mfr # GCM31CC72A225KE02L -> (none); Mouser https://www.mouser.com/en/ProductDetail/Murata-Electronics/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 -> (none); Mouser # 81-GCM31CC72A225KE2L -> (none); Mouser Lifecycle Unknown -> (none); Mouser Price Breaks (Raw) 1:0.63|10:0.31|100:0.272|500:0.233|1000:0.218|2000:0.192|40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 -> (none); Mouser Qty/Price 1:$0.63 | 10:$0.31 | 100:$0.27 | 500:$0.23 -> (none); Mouser Stock 26577 In Stock -> (none); Mouser Stock Qty 26577 -> (none); Vendor Description Multilayer Ceramic Capacitors MLCC - SMD/SMT 2.2 uF 100 VDC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 -> (none)
- C20, C22, C3, C4, C5, C8: Last Checked 2026-08-09T03:01:00.990148+00:00 -> (none); Mfr KEMET -> (none); Mfr # C0402C104K4RACAUTO7411 -> (none); Mouser https://www.mouser.com/en/ProductDetail/KEMET/C0402C104K4RA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 -> (none); Mouser # 80-C0402C104K4RAUTLR -> (none); Mouser Lifecycle Unknown -> (none); Mouser Price Breaks (Raw) 1:0.13|10:0.054|100:0.032|500:0.025|1000:0.024|50000:0.024 -> (none); Mouser Qty/Price 1:$0.13 | 10:$0.05 | 100:$0.03 | 500:$0.03 -> (none); Mouser Stock 80862 In Stock -> (none); Mouser Stock Qty 80862 -> (none); Vendor Description Multilayer Ceramic Capacitors MLCC - SMD/SMT 16V 0.1uF X7R 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 -> (none)
- C21: Last Checked 2026-08-09T03:01:00.990148+00:00 -> (none); Mfr YAGEO -> (none); Mfr # AC0805KFX7R8BB474 -> (none); Mouser https://www.mouser.com/en/ProductDetail/YAGEO/AC0805KFX7R8B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 -> (none); Mouser # 603-AC805KFX7R8BB474 -> (none); Mouser Lifecycle Unknown -> (none); Mouser Price Breaks (Raw) 1:0.25|10:0.106|100:0.093|500:0.072|1000:0.066|2500:0.059|5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 -> (none); Mouser Qty/Price 1:$0.25 | 10:$0.11 | 100:$0.09 | 500:$0.07 -> (none); Mouser Stock 9946 In Stock -> (none); Mouser Stock Qty 9946 -> (none); Vendor Description Multilayer Ceramic Capacitors MLCC - SMD/SMT 25V 0.47uF X7R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 -> (none)
- C23: Last Checked 2026-08-09T03:01:00.990148+00:00 -> (none); Mfr KYOCERA AVX -> (none); Mfr # 08051C474K4T2A -> (none); Mouser https://www.mouser.com/en/ProductDetail/KYOCERA-AVX/08051C4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 -> (none); Mouser # 581-08051C474K4T2A -> (none); Mouser Lifecycle Unknown -> (none); Mouser Price Breaks (Raw) 1:0.31|10:0.299|2000:0.299|4000:0.207 -> (none); Mouser Qty/Price 1:$0.31 | 10:$0.30 | 2000:$0.30 | 4000:$0.21 -> (none); Mouser Stock 20923 In Stock -> (none); Mouser Stock Qty 20923 -> (none); Vendor Description Multilayer Ceramic Capacitors MLCC - SMD/SMT KAM21KR72A474K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 -> (none)
- C6: Last Checked 2026-08-09T03:01:00.990148+00:00 -> (none); Mfr Murata Electronics -> (none); Mfr # GRM32ER71E226ME15L -> (none); Mouser https://www.mouser.com/en/ProductDetail/Murata-Electronics/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 -> (none); Mouser # 81-GRM32ER71E226ME5L -> (none); Mouser Lifecycle End of Life -> (none); Mouser Price Breaks (Raw) 1:0.78|10:0.376|100:0.34|500:0.28|1000:0.247|2000:0.226 -> (none); Mouser Qty/Price 1:$0.78 | 10:$0.38 | 100:$0.34 | 500:$0.28 -> (none); Mouser Stock 1646 In Stock -> (none); Mouser Stock Qty 1646 -> (none); Vendor Description Multilayer Ceramic Capacitors MLCC - SMD/SMT 22 uF 25 VDC 2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 -> (none)
- C9: Last Checked 2026-08-09T03:01:00.990148+00:00 -> (none); Mfr TDK -> (none); Mfr # CGA4J3X7R1H155K125AB -> (none); Mouser https://www.mouser.com/en/ProductDetail/TDK/CGA4J3X7R1H155K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 -> (none); Mouser # 810-CGA4J3X7R1H155KB -> (none); Mouser Lifecycle Unknown -> (none); Mouser Price Breaks (Raw) 1:0.37|10:0.165|100:0.147|500:0.116|1000:0.107|2000:0.095|4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 -> (none); Mouser Qty/Price 1:$0.37 | 10:$0.17 | 100:$0.15 | 500:$0.12 -> (none); Mouser Stock 7563 In Stock -> (none); Mouser Stock Qty 7563 -> (none); Vendor Description Multilayer Ceramic Capacitors MLCC - SMD/SMT CGA 0805 50V 1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 -> (none)
- D1: Last Checked 2026-08-09T03:01:00.990148+00:00 -> (none); Mfr Littelfuse -> (none); Mfr # SMAJ40A -> (none); Mouser https://www.mouser.com/en/ProductDetail/Littelfuse/SMAJ40A?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 -> (none); Mouser # 576-SMAJ40A -> (none); Mouser Lifecycle Unknown -> (none); Mouser Price Breaks (Raw) 1:0.38|10:0.208|100:0.175|500:0.135|1000:0.117|2500:0.098|5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 -> (none); Mouser Qty/Price 1:$0.38 | 10:$0.21 | 100:$0.17 | 500:$0.14 -> (none); Mouser Stock 42488 In Stock -> (none); Mouser Stock Qty 42488 -> (none); Vendor Description ESD Protection Diodes / TVS Diodes 400W 40V 5% Uni-Directio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 -> (none)
- D10: DigiKey https://www.digikey.com/en/products/detail/yageo/ES1B/20415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 -> (none); DigiKey # 13-ES1BCT-ND -> (none); DigiKey Lifecycle Active -> (none); DigiKey Price Breaks (Raw) 1:0.34|10:0.208|50:0.149|100:0.1298|500:0.09588 -> (none); DigiKey Qty/Price 1:$0.34 | 10:$0.21 | 50:$0.15 | 100:$0.13 -> (none); DigiKey Stock 1305 in stock -> (none); DigiKey Stock Qty 1305 -> (none); Last Checked 2026-08-09T03:01:00.990148+00:00 -> (none); Mfr YAGEO -> (none); Mfr # ES1B -> (none); Vendor Description Diode 100 V 1A Surface Mount DO-214AC (SMA) -> (none)
- D11, D9: DigiKey https://www.digikey.com/en/products/detail/diotec-semicondu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 -> (none); DigiKey # 4878-1N4148WGWCT-ND -> (none); DigiKey Lifecycle Active -> (none); DigiKey Price Breaks (Raw) 1:0.1|10:0.057|50:0.04|100:0.0346|500:0.02478 -> (none); DigiKey Qty/Price 1:$0.10 | 10:$0.06 | 50:$0.04 | 100:$0.03 -> (none); DigiKey Stock 24163 in stock -> (none); DigiKey Stock Qty 24163 -> (none); Last Checked 2026-08-09T03:01:00.990148+00:00 -> (none); Mfr Diotec Semiconductor -> (none); Mfr # 1N4148WGW -> (none); Vendor Description Diode 75 V 150mA Surface Mount SOD-123 -> (none)
- D12, D13: DigiKey https://www.digikey.com/en/products/detail/taiwan-semicondu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 -> (none); DigiKey # 1801-TSSA5U60HCT-ND -> (none); DigiKey Lifecycle Active -> (none); DigiKey Price Breaks (Raw) 1:0.7|10:0.432|50:0.3144|100:0.2762|500:0.20876 -> (none); DigiKey Qty/Price 1:$0.70 | 10:$0.43 | 50:$0.31 | 100:$0.28 -> (none); DigiKey Stock 13127 in stock -> (none); DigiKey Stock Qty 13127 -> (none); Last Checked 2026-08-09T03:01:00.990148+00:00 -> (none); Mfr Taiwan Semiconductor Corporation -> (none); Mfr # TSSA5U60H -> (none); Vendor Description Diode 60 V 5A Surface Mount DO-214AC (SMA) -> (none)
- D14, D15: DigiKey https://www.digikey.com/en/products/detail/rohm-semiconduct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 -> (none); DigiKey # 846-SMLMN2ECTT86CCT-ND -> (none); DigiKey Lifecycle Active -> (none); DigiKey Price Breaks (Raw) 1:0.75|10:0.521|100:0.3792|500:0.31586|1000:0.29509 -> (none); DigiKey Qty/Price 1:$0.75 | 10:$0.52 | 100:$0.38 | 500:$0.32 -> (none); DigiKey Stock 804 in stock -> (none); DigiKey Stock Qty 804 -> (none); Last Checked 2026-08-09T03:01:00.990148+00:00 -> (none); Mfr Rohm Semiconductor -> (none); Mfr # SMLMN2ECTT86C -> (none); Vendor Description Green 527nm LED Indication - Discrete 3V 0805 (2012 Metric) -> (none)
- D2: DigiKey https://www.digikey.com/en/products/detail/würth-elektronik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 -> (none); DigiKey # 732-SMAJ24ACT-ND -> (none); DigiKey Lifecycle Active -> (none); DigiKey Price Breaks (Raw) 1:0.29|10:0.269|100:0.241|500:0.21 -> (none); DigiKey Qty/Price 1:$0.29 | 10:$0.27 | 100:$0.24 | 500:$0.21 -> (none); DigiKey Stock 10565 in stock -> (none); DigiKey Stock Qty 10565 -> (none); Last Checked 2026-08-09T03:01:00.990148+00:00 -> (none); Mfr Würth Elektronik -> (none); Mfr # SMAJ24A -> (none); Mouser https://www.mouser.com/en/ProductDetail/YAGEO/SMAJ24A-TR7?q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 -> (none); Mouser # 603-SMAJ24A/TR7 -> (none); Mouser Lifecycle Unknown -> (none); Mouser Price Breaks (Raw) 1:0.37|10:0.161|100:0.141|500:0.104|1000:0.092|2000:0.068|5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 -> (none); Mouser Qty/Price 1:$0.37 | 10:$0.16 | 100:$0.14 | 500:$0.10 -> (none); Mouser Stock 1540 In Stock -> (none); Mouser Stock Qty 1540 -> (none); Vendor Description 38.9V Clamp 10.3A Ipp Tvs Diode Surface Mount DO-214AC -> (none)
- D3, D8: DigiKey https://www.digikey.com/en/products/detail/rohm-semiconduct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 -> (none); DigiKey # 846-SMLMN2ECTT86CTR-ND -> (none); DigiKey Lifecycle Active -> (none); DigiKey Price Breaks (Raw) 3000:0.26838|6000:0.25478|9000:0.24781|15000:0.23994|21000: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 -> (none); DigiKey Qty/Price 3000:$0.27 | 6000:$0.25 | 9000:$0.25 | 15000:$0.24 -> (none); DigiKey Stock 804 in stock -> (none); DigiKey Stock Qty 804 -> (none); Last Checked 2026-08-09T03:01:00.990148+00:00 -> (none); Mfr ROHM Semiconductor -> (none); Mfr # SMLMN2ECTT86C -> (none); Mouser https://www.mouser.com/en/ProductDetail/ROHM-Semiconductor/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 -> (none); Mouser # 755-SMLMN2ECTT86C -> (none); Mouser Lifecycle Unknown -> (none); Mouser Price Breaks (Raw) 1:0.73|10:0.506|100:0.369|500:0.308|1000:0.288|3000:0.264|6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 -> (none); Mouser Qty/Price 1:$0.73 | 10:$0.51 | 100:$0.37 | 500:$0.31 -> (none); Mouser Stock 724 In Stock -> (none); Mouser Stock Qty 724 -> (none); Vendor Description Single Color LEDs Add PTC 5-0617-50 AECQ-102 -> (none)
- D4: Last Checked 2026-08-09T03:01:00.990148+00:00 -> (none); Mfr Diodes Incorporated -> (none); Mfr # DDZ9699T-7 -> (none); Mouser https://www.mouser.com/en/ProductDetail/Diodes-Incorporated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 -> (none); Mouser # 621-DDZ9699T-7 -> (none); Mouser Lifecycle Unknown -> (none); Mouser Price Breaks (Raw) 1:0.51|10:0.235|100:0.193|500:0.174|1000:0.158|3000:0.158 -> (none); Mouser Qty/Price 1:$0.51 | 10:$0.23 | 100:$0.19 | 500:$0.17 -> (none); Mouser Stock 7675 In Stock -> (none); Mouser Stock Qty 7675 -> (none); Vendor Description Zener Diodes 150MW 12V -> (none)
- D5: Last Checked 2026-08-09T03:01:00.990148+00:00 -> (none); Mfr ROHM Semiconductor -> (none); Mfr # SML-H12U8TT86C -> (none); Mouser https://www.mouser.com/en/ProductDetail/ROHM-Semiconductor/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 -> (none); Mouser # 755-SML-H12U8TT86C -> (none); Mouser Lifecycle Unknown -> (none); Mouser Price Breaks (Raw) 1:0.31|10:0.213|100:0.15|500:0.122|1000:0.11|3000:0.099|600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 -> (none); Mouser Qty/Price 1:$0.31 | 10:$0.21 | 100:$0.15 | 500:$0.12 -> (none); Mouser Stock 12678 In Stock -> (none); Mouser Stock Qty 12678 -> (none); Vendor Description Single Color LEDs The factory is currently not accepting or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 -> (none)
- D6, D7: Last Checked 2026-08-09T03:01:00.990148+00:00 -> (none); Mfr Panjit -> (none); Mfr # BAT54C-AU_R1_000A1 -> (none); Mouser https://www.mouser.com/en/ProductDetail/Panjit/BAT54C-AU_R1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 -> (none); Mouser # 241-BAT54C-AUR1000A1 -> (none); Mouser Lifecycle Unknown -> (none); Mouser Price Breaks (Raw) 1:0.19|10:0.118|100:0.074|500:0.06|1000:0.052|3000:0.045|60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 -> (none); Mouser Qty/Price 1:$0.19 | 10:$0.12 | 100:$0.07 | 500:$0.06 -> (none); Mouser Stock 3073 In Stock -> (none); Mouser Stock Qty 3073 -> (none); Vendor Description Schottky Diodes & Rectifiers 30V,Schottky,SOT-23,0.2A -> (none)
- IC1: DigiKey https://www.digikey.com/en/products/detail/texas-instrument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 -> (none); DigiKey # 296-23126-1-ND -> (none); DigiKey Lifecycle Active -> (none); DigiKey Price Breaks (Raw) 1:2.33|10:1.727|25:1.5756|100:1.4094|250:1.33024|500:1.29132 -> (none); DigiKey Qty/Price 1:$2.33 | 10:$1.73 | 25:$1.58 | 100:$1.41 -> (none); DigiKey Stock 0 in stock -> (none); DigiKey Stock Qty 0 -> (none); Last Checked 2026-08-09T03:01:00.990148+00:00 -> (none); Mfr Texas Instruments -> (none); Mfr # TPS3808G50QDBVRQ1 -> (none); Vendor Description Supervisor Open Drain or Open Collector 1 Channel SOT-23-6 -> (none)
- J1, J3, JP1: Last Checked 2026-08-09T03:15:47.868936+00:00 -> (none)
- J4: DigiKey https://www.digikey.com/en/products/detail/amphenol-cs-fci/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 -> (none); DigiKey Lifecycle Active -> (none); DigiKey Price Breaks (Raw) 1:2.67|10:2.271|100:1.9297 -> (none); DigiKey Qty/Price 1:$2.67 | 10:$2.27 | 100:$1.93 -> (none); DigiKey Stock 8712 in stock -> (none); DigiKey Stock Qty 8712 -> (none); Last Checked 2026-08-09T03:01:00.990148+00:00 -> (none); Mfr Amphenol ICC (FCI) -> Amphenol ICC; Vendor Description 20 Position Receptacle Connector 0.050" (1.27mm) Surface Mo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 -> (none)
- L1: DigiKey https://www.digikey.com/en/products/detail/bourns-inc/SRR12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 -> (none); DigiKey # SRR1260A-2R2YCT-ND -> (none); DigiKey Lifecycle Active -> (none); DigiKey Price Breaks (Raw) 1:1.3|10:1.066|25:0.986|50:0.9294|100:0.8763|250:0.81072 -> (none); DigiKey Qty/Price 1:$1.30 | 10:$1.07 | 25:$0.99 | 50:$0.93 -> (none); DigiKey Stock 262 in stock -> (none); DigiKey Stock Qty 262 -> (none); Last Checked 2026-08-09T03:01:00.990148+00:00 -> (none); Mfr Bourns Inc. -> (none); Mfr # SRR1260A-2R2Y -> (none); Vendor Description 2.2 µH Shielded Drum Core, Wirewound Inductor 8.2 A 10.5mOh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 -> (none)
- Q1: DigiKey https://www.digikey.com/en/products/detail/nexperia-usa-inc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 -> (none); DigiKey # 1727-BUK7J2R4-80MXCT-ND -> (none); DigiKey Lifecycle Active -> (none); DigiKey Price Breaks (Raw) 1:3.61|10:2.356|50:1.8138|100:1.6392|500:1.3331 -> (none); DigiKey Qty/Price 1:$3.61 | 10:$2.36 | 50:$1.81 | 100:$1.64 -> (none); DigiKey Stock 1407 in stock -> (none); DigiKey Stock Qty 1407 -> (none); Last Checked 2026-08-09T03:01:00.990148+00:00 -> (none); Mfr Nexperia USA Inc. -> (none); Mfr # BUK7J2R4-80MX -> (none); Vendor Description N-Channel 80 V 231A (Ta) 294W (Ta) Surface Mount LFPAK56, P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 -> (none)
- Q2, Q3, Q4: DigiKey https://www.digikey.com/en/products/detail/nexperia-usa-inc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 -> (none); DigiKey # 1727-1142-1-ND -> (none); DigiKey Lifecycle Active -> (none); DigiKey Price Breaks (Raw) 1:0.19|10:0.119|50:0.0848|100:0.0735|500:0.05348 -> (none); DigiKey Qty/Price 1:$0.19 | 10:$0.12 | 50:$0.08 | 100:$0.07 -> (none); DigiKey Stock 74456 in stock -> (none); DigiKey Stock Qty 74456 -> (none); Last Checked 2026-08-09T03:01:00.990148+00:00 -> (none); Mfr Nexperia USA Inc. -> (none); Mfr # BSS138P,215 -> (none); Vendor Description N-Channel 60 V 360mA (Ta) 350mW (Ta), 1.14W (Tc) Surface Mo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 -> (none)
- R1, R16, R2, R30: DigiKey https://www.digikey.com/en/products/detail/vishay-dale/CRCW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 -> (none); DigiKey # 541-100KLCT-ND -> (none); DigiKey Lifecycle Active -> (none); DigiKey Price Breaks (Raw) 1:0.1|10:0.032|25:0.0236|50:0.0192|100:0.0157|250:0.01228|5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 -> (none); DigiKey Qty/Price 1:$0.10 | 10:$0.03 | 25:$0.02 | 50:$0.02 -> (none); DigiKey Stock 4115632 in stock -> (none); DigiKey Stock Qty 4115632 -> (none); Last Checked 2026-08-09T03:01:00.990148+00:00 -> (none); Mfr Vishay Dale -> (none); Mfr # CRCW0402100KFKED -> (none); Mouser https://www.mouser.com/en/ProductDetail/Vishay/CRCW0402100K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 -> (none); Mouser # 71-CRCW0402-100K-E3 -> (none); Mouser Lifecycle Unknown -> (none); Mouser Price Breaks (Raw) 1:0.1|10:0.02|100:0.016|250:0.013|500:0.011|1000:0.009|5000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 -> (none); Mouser Qty/Price 1:$0.10 | 10:$0.02 | 100:$0.02 | 250:$0.01 -> (none); Mouser Replacement 71-CRCW0402-100K -> (none); Mouser Stock 2923962 In Stock -> (none); Mouser Stock Qty 2923962 -> (none); Vendor Description 100 kOhms ±1% 0.063W, 1/16W Chip Resistor 0402 (1005 Metric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 -> (none)
- R10, R13, R34: DigiKey https://www.digikey.com/en/products/detail/vishay-dale/CRCW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 -> (none); DigiKey # 541-1.00KCCT-ND -> (none); DigiKey Lifecycle Active -> (none); DigiKey Price Breaks (Raw) 1:0.1|10:0.044|25:0.0332|50:0.0272|100:0.0225|250:0.01796|5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 -> (none); DigiKey Qty/Price 1:$0.10 | 10:$0.04 | 25:$0.03 | 50:$0.03 -> (none); DigiKey Stock 1347365 in stock -> (none); DigiKey Stock Qty 1347365 -> (none); Last Checked 2026-08-09T03:01:00.990148+00:00 -> (none); Mfr Vishay Dale -> (none); Mfr # CRCW08051K00FKEA -> (none); Mouser https://www.mouser.com/en/ProductDetail/Vishay/CRCW08051K00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 -> (none); Mouser # 71-CRCW0805-1.0K-E3 -> (none); Mouser Lifecycle Unknown -> (none); Mouser Price Breaks (Raw) 1:0.1|10:0.028|100:0.023|250:0.018|500:0.016|1000:0.014|500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 -> (none); Mouser Qty/Price 1:$0.10 | 10:$0.03 | 100:$0.02 | 250:$0.02 -> (none); Mouser Replacement 71-CRCW0805-1.0K -> (none); Mouser Stock 468345 In Stock -> (none); Mouser Stock Qty 468345 -> (none); Vendor Description 1 kOhms ±1% 0.125W, 1/8W Chip Resistor 0805 (2012 Metric) A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 -> (none)
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